File: board/board.kicad_pcb (KiCad board)
At the start: 4 copper layers, 68.6 x 58.4 mm, 81 parts, among them J1 Molex Picoblade, J2 Conn_ARM_JTAG_SWD_10, J3 USB_B_Micro, J4 Conn_01x04_Male, J5 Screw_Terminal_01x02, J6 Conn_01x06_Male, Q1 FDV305N, Q2 FDV305N, Q3 FDV305N, Q5 Find one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

Commit message: Push
Parts:
- removed C31: 1u, Capacitor_SMD:C_0402_1005Metric
- removed C32: 100n, Capacitor_SMD:C_0402_1005Metric
- removed Q5: Find one, Package_TO_SOT_SMD:SOT-23
- removed R16: 100, Resistor_SMD:R_0402_1005Metric
- removed U4: UCC2751x, Package_TO_SOT_SMD:SOT-23-5
- added D3: B5817W, Diode_SMD:D_0805_2012Metric, F.Cu at (77.9, 92.8)
- added D4: LED, LED_SMD:LED_0603_1608Metric, F.Cu at (81.6, 97.7)
- added J7: Conn_01x07_Female, Connector_PinSocket_2.54mm:PinSocket_1x07_P2.54mm_Vertical, F.Cu at (96.8, 126.2)
- added J9: Screw_Terminal_01x02, TerminalBlock_Phoenix:TerminalBlock_Phoenix_PT-1,5-2-5.0-H_1x02_P5.00mm_Horizontal, F.Cu at (83.5, 87.0)
- added R1: 619k, Resistor_SMD:R_0402_1005Metric, F.Cu at (78.1, 125.6)
- added R2: 137k, Resistor_SMD:R_0402_1005Metric, F.Cu at (78.6, 124.0)
- added SW1: SW_SPDT, Button_Switch_SMD:SW_SPDT_PCM12, F.Cu at (127.5, 123.3)
- added TP1: TestPoint, TestPoint:TestPoint_Pad_D1.0mm, F.Cu at (106.7, 109.7)
- added TP2: TestPoint, TestPoint:TestPoint_Pad_D1.0mm, F.Cu at (68.0, 96.8)
- added TP4: TestPoint, TestPoint:TestPoint_Pad_D1.0mm, F.Cu at (64.5, 92.5)
- added U3: DRV104PWPR, DRV104PWPR:IC_TPS27S100BPWPR, F.Cu at (76.5, 98.5)
- C15: value 22u -> 10u
- C16: value 10u -> 1u; footprint Capacitor_SMD:C_0603_1608Metric -> Capacitor_SMD:C_0402_1005Metric
- C18: value 100n -> 22p; footprint Capacitor_SMD:C_0603_1608Metric -> Capacitor_SMD:C_0402_1005Metric
- C21: value 1u -> 22u; footprint Capacitor_SMD:C_0603_1608Metric -> Capacitor_SMD:C_0402_1005Metric
- C22: value 100n -> 22u; footprint Capacitor_SMD:C_0603_1608Metric -> Capacitor_SMD:C_0402_1005Metric
- C23: footprint Capacitor_SMD:C_0603_1608Metric -> Capacitor_SMD:C_0402_1005Metric
- C24: value 22u -> 22p; footprint Capacitor_SMD:C_0603_1608Metric -> Capacitor_SMD:C_0402_1005Metric
- C30: value 100n -> 470p
- F1: value 300mA -> 0ZCJ0050AF2E
- L1: value 4u7 -> 2u7
- L2: value 2u2 -> 3u3
- Q1, Q2, Q3: footprint SOT95P240X111-3N -> FDV305N:SOT95P240X111-3N
- R10: value 73k2 -> 619k; footprint Resistor_SMD:R_0603_1608Metric -> Resistor_SMD:R_0402_1005Metric
- R11: value 22k1 -> 84k5; footprint Resistor_SMD:R_0603_1608Metric -> Resistor_SMD:R_0402_1005Metric
- R13: footprint Resistor_SMD:R_0402_1005Metric -> Resistor_SMD:R_0603_1608Metric
- R5: value 124k -> 10k
- R6: value 22k1 -> 5k6
- U2: value TPS542941 -> LTC3622-23_5; footprint Package_SO:HTSSOP-16-1EP_4.4x5mm_P0.65mm_EP3.4x5mm_Mask2.46x2.31mm_ThermalVias -> Package_SO:MSOP-16-1EP_3x4mm_P0.5mm_EP1.65x2.85mm_ThermalVias
- moved R5 49.9 mm to (121.8, 123.1), turned to 0 degrees
- moved R6 29.4 mm to (81.5, 100.3), turned to 0 degrees
- moved C30 28.2 mm to (87.9, 99.9), turned to 0 degrees
- moved D1 21.5 mm to (106.4, 100.1)
- moved R4 21.5 mm to (106.4, 101.7)
- moved C23 20.3 mm to (85.0, 100.0), turned to 0 degrees
- moved C26 18.8 mm to (87.2, 120.4)
- moved C25 18.8 mm to (87.3, 121.5)
- moved R15 16.0 mm to (115.1, 111.4), turned to 270 degrees
- moved R10 13.2 mm to (78.4, 121.4), turned to 90 degrees
- moved R17 12.4 mm to (121.1, 117.8)
- moved R11 12.1 mm to (77.3, 122.0), turned to 270 degrees
- moved L2 12.0 mm to (76.1, 120.2)
- moved R13 10.3 mm to (85.6, 97.7)
- moved C24 9.10 mm to (79.4, 121.4), turned to 270 degrees
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Connections:
- C15 pad 1: +5V -> +12V
- C16 pad 1: BUCK_IN -> INTVCC
- C18 pad 1: VBST1 -> +3V3
- C18 pad 2: SW1 -> FB2
- C20 pad 1: BUCK_IN -> +12V
- C21 pad 1: Net-(C21-Pad1) -> +3V3
- C22 pad 1: VBST2 -> +5V
- C22 pad 2: SW2 -> GND
- C23 pad 1: BUCK_IN -> GND
- C23 pad 2: GND -> +12V
- C24 pad 1: +3V3 -> +5V
- C24 pad 2: GND -> FB1
- C30 pad 1: +3V3 -> CBOOT
- C30 pad 2: GND -> DRVOUT
- F1 pad 2: +UCC_VDD -> +12V
- FB2 pad 1: BUCK_IN -> +12V
- J5 pad 1: +UCC_VDD -> GND
- J5 pad 2: GND -> +12V
- L1 pad 1: +5V -> SW2
- L1 pad 2: SW1 -> +3V3
- L2 pad 1: SW2 -> SW1
- L2 pad 2: +3V3 -> +5V
- R10 pad 1: VFB2 -> FB1
- R10 pad 2: +3V3 -> +5V
- R11 pad 2: VFB2 -> FB1
- R13 pad 1: UCC_EN -> GND
- R13 pad 2: +UCC_VDD -> Net-(R13-Pad2)
- R5 pad 1: VFB1 -> Net-(R5-Pad1)
- R5 pad 2: +5V -> BOOT0
- R6 pad 1: GND -> Net-(D4-Pad2)
- R6 pad 2: VFB1 -> +12V
- U1 pad 10: LCD_DB2 -> Net-(U1-Pad10)
- U1 pad 11: LCD_DB3 -> Net-(U1-Pad11)
- U1 pad 24: Net-(U1-Pad24) -> LCD_DB0
- U1 pad 25: Net-(U1-Pad25) -> LCD_DB1
- U1 pad 26: Net-(U1-Pad26) -> LCD_DB2
- U1 pad 28: Net-(U1-Pad28) -> LCD_DB3
- U1 pad 33: SPI2_!CS -> Net-(U1-Pad33)
- U1 pad 37: FLASH_!WP -> Net-(U1-Pad37)
- U1 pad 38: FLASH_!HOLD -> SPI2_!CS
- U1 pad 39: Net-(U1-Pad39) -> FLASH_!WP
- U1 pad 40: Net-(U1-Pad40) -> FLASH_!HOLD
- U1 pad 8: LCD_DB0 -> Net-(U1-Pad8)
- U1 pad 9: LCD_DB1 -> Net-(U1-Pad9)
- U2 pad 1: BUCK_IN -> +12V
- U2 pad 10: VFB2 -> +12V
- U2 pad 11: Net-(U2-Pad11) -> FB2
- U2 pad 12: EN2_IN -> INTVCC
- U2 pad 13: GND -> FB1
- U2 pad 14: SW2 -> +12V
- U2 pad 15: VBST2 -> GND
- U2 pad 16: BUCK_IN -> SW1
- U2 pad 2: VBST1 -> +12V
- U2 pad 3: SW1 -> Net-(U2-Pad3)
- U2 pad 4: GND -> INTVCC
- U2 pad 5: EN1_IN -> GND
- U2 pad 7: VFB1 -> GND
- U2 pad 8: GND -> +12V
- U2 pad 9: Net-(C21-Pad1) -> SW2
Routing:
- net NRST: track 1.73 -> 31.6 mm, vias 0 -> 2
- net SPI2_MISO: track 0.00 -> 28.0 mm, vias 0 -> 2
- net FLASH_!WP: track 0.00 -> 20.2 mm
- net FLASH_!HOLD: track 0.00 -> 18.1 mm
- net SWO: track 0.00 -> 17.2 mm, vias 0 -> 2
- net SWDCLK: track 0.00 -> 14.9 mm
- net GND: track 16.7 -> 30.8 mm, vias 2 -> 15
- net SPI2_CLK: track 0.00 -> 11.7 mm
- net SPI2_MOSI: track 0.00 -> 11.6 mm
- net +12V: track 0.00 -> 9.15 mm, vias 0 -> 5
- net FB2: track 0.00 -> 6.05 mm
- net INTVCC: track 0.00 -> 5.59 mm, vias 0 -> 1
- net SPI2_!CS: track 16.2 -> 20.7 mm
- net FB1: track 0.00 -> 3.65 mm
- net +3V3: track 15.6 -> 18.8 mm, vias 0 -> 4
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- added copper zone on In2.Cu, net +12V
- added copper zone on F.Cu, net +3V3
- added copper zone on In2.Cu, net +3V3
- added copper zone on F.Cu, net +5V
- added copper zone on In2.Cu, net +5V
- added copper zone on F.Cu, net SW1
- added copper zone on F.Cu, net SW2
