File: board/board.sch (KiCad schematic (older format))
At the start: 46 parts, among them Q2 Q_NMOS_GDS, Q3 Q_NMOS_GDS, Q4 Q_NMOS_GDS, U2 TPS542941, Y1 16MHz

Commit message: Update
Parts:
- removed D2: LED_RGB, LED_SMD:LED_RGB_1210, symbol Device:LED_RGB
- removed Q2, Q3, Q4: Q_NMOS_GDS, Package_TO_SOT_SMD:SOT-23, symbol Device:Q_NMOS_GDS
- added D2: ASMB-KTF0-0A306, LED_SMD:LED_ASMB-KTF0-0A306, symbol ASMB-KTF0-0A306:ASMB-KTF0-0A306
- added Q1, Q2, Q3: FDV305N, SOT95P240X111-3N, symbol FDV305N:FDV305N
- gave numbers to parts that had none: 1
Connections:
- wire segments 147 -> 145
Other:
- note added: "B"
- note added: "G"
- note added: "R"
- note removed: "Find RGB\n"
- moved on the sheet: C19
Changed lines of the file:
@@
 Wire Notes Line
 	6800 7350 4500 7350
-Text GLabel 5850 6550 0    50   Input ~ 0
+Text GLabel 5950 6650 0    50   Input ~ 0
 TIM4_CH3
-Text GLabel 5400 6850 0    50   Input ~ 0
+Text GLabel 5500 6950 0    50   Input ~ 0
 TIM4_CH2
-$Comp
-L Device:Q_NMOS_GDS Q2
-U 1 1 60C23A9D
-P 5200 6550
-F 0 "Q2" H 5400 6700 50  0000 L CNN
-F 1 "Q_NMOS_GDS" H 5100 6600 50  0000 L CNN
-F 2 "Package_TO_SOT_SMD:SOT-23" H 5400 6650 50  0001 C CNN
-F 3 "~" H 5200 6550 50  0001 C CNN
-	1    5200 6550
-	1    0    0    -1
-$EndComp
 Wire Wire Line
 	5700 7200 5700 7150
@@
 Wire Wire Line
 	5700 7150 5300 7150
-Text GLabel 5000 6550 0    50   Input ~ 0
+Text GLabel 5100 6650 0    50   Input ~ 0
 TIM4_CH1
 Wire Wire Line
@@
 Wire Wire Line
 	6150 6350 6150 6300
-$Comp
-L Device:Q_NMOS_GDS Q3
-U 1 1 60C22167
-P 5600 6850
-F 0 "Q3" H 5804 6896 50  0000 L CNN
-F 1 "Q_NMOS_GDS" H 5804 6805 50  0000 L CNN
-F 2 "Package_TO_SOT_SMD:SOT-23" H 5800 6950 50  0001 C CNN
-F 3 "~" H 5600 6850 50  0001 C CNN
-	1    5600 6850
-	1    0    0    -1
-$EndComp
-$Comp
-L Device:Q_NMOS_GDS Q4
-U 1 1 60C1AFA5
-P 6050 6550
-F 0 "Q4" H 6250 6700 50  0000 L CNN
-F 1 "Q_NMOS_GDS" H 6250 6600 50  0000 L CNN
-F 2 "Package_TO_SOT_SMD:SOT-23" H 6250 6650 50  0001 C CNN
-F 3 "~" H 6050 6550 50  0001 C CNN
-	1    6050 6550
-	1    0    0    -1
-$EndComp
-Connection ~ 5900 5550
-Wire Wire Line
-	5900 5650 5900 5550
-Wire Wire Line
-	5500 5550 5700 5550
-Wire Wire Line
-	5500 5650 5500 5550
-Wire Wire Line
-	5700 5500 5700 5550
-Connection ~ 5700 5550
-Wire Wire Line
-	5900 5550 5700 5550
-Wire Wire Line
-	6150 5550 6100 5550
 $Comp
 L power:GND #PWR022
 U 1 1 60BEDB34
-P 6150 5550
-F 0 "#PWR022" H 6150 5300 50  0001 C CNN
-F 1 "GND" H 6155 5377 50  0000 C CNN
-F 2 "" H 6150 5550 50  0001 C CNN
-F 3 "" H 6150 5550 50  0001 C CNN
-	1    6150 5550
+P 5800 5550
+F 0 "#PWR022" H 5800 5300 50  0001 C CNN
+F 1 "GND" H 5805 5377 50  0000 C CNN
+F 2 "" H 5800 5550 50  0001 C CNN
+F 3 "" H 5800 5550 50  0001 C CNN
+	1    5800 5550
 	0    -1   -1   0
 $EndComp
-Wire Wire Line
-	5700 5550 5700 5650
 $Comp
 L power:+3V3 #PWR020
 U 1 1 60BE178F
-P 5700 5500
-F 0 "#PWR020" H 5700 5350 50  0001 C CNN
-F 1 "+3V3" H 5715 5673 50  0000 C CNN
-F 2 "" H 5700 5500 50  0001 C CNN
-F 3 "" H 5700 5500 50  0001 C CNN
-	1    5700 5500
+P 5500 5500
+F 0 "#PWR020" H 5500 5350 50  0001 C CNN
+F 1 "+3V3" H 5515 5673 50  0000 C CNN
+F 2 "" H 5500 5500 50  0001 C CNN
+F 3 "" H 5500 5500 50  0001 C CNN
+	1    5500 5500
 	1    0    0    -1
 $EndComp
@@
 L Device:C_Small C19
 U 1 1 60BE1075
-P 6000 5550
-F 0 "C19" V 5900 5600 50  0000 L CNN
-F 1 "10u" V 6100 5600 50  0000 L CNN
-F 2 "Capacitor_SMD:C_0603_1608Metric" H 6000 5550 50  0001 C CNN
-F 3 "~" H 6000 5550 50  0001 C CNN
-	1    6000 5550
+P 5700 5550
+F 0 "C19" V 5600 5600 50  0000 L CNN
+F 1 "10u" V 5800 5600 50  0000 L CNN
+F 2 "Capacitor_SMD:C_0603_1608Metric" H 5700 5550 50  0001 C CNN
+F 3 "~" H 5700 5550 50  0001 C CNN
+	1    5700 5550
 	0    1    1    0
 $EndComp
@@
 Wire Wire Line
 	5500 6050 5300 6050
-Wire Wire Line
-	5700 6050 5700 6100
 Wire Wire Line
 	6150 6050 6150 6100
@@
 	1    5300 6200
 	-1   0    0    1
-$EndComp
-$Comp
-L Device:LED_RGB D2
-U 1 1 60BB57C8
-P 5700 5850
-F 0 "D2" V 5746 5520 50  0000 R CNN
-F 1 "LED_RGB" V 5655 5520 50  0000 R CNN
-F 2 "LED_SMD:LED_RGB_1210" H 5700 5800 50  0001 C CNN
-F 3 "~" H 5700 5800 50  0001 C CNN
-	1    5700 5850
-	0    -1   -1   0
 $EndComp
 Wire Notes Line
@@
 Wire Wire Line
 	4800 1950 4800 2100
-Text Notes 6650 5550 0    98   ~ 20
-Find RGB\n
 Text GLabel 1700 5100 0    50   Input ~ 0
 USART3_TX
@@
 USART3_RX
 $Comp
-L MCU_ST_STM32F4:STM32F405RGTx U?
+L MCU_ST_STM32F4:STM32F405RGTx U1
 U 1 1 60C86C3C
 P 2400 4000
-F 0 "U?" H 2850 5800 50  0000 C CNN
+F 0 "U1" H 2850 5800 50  0000 C CNN
 F 1 "STM32F405RGTx" H 2950 2150 50  0000 C CNN
 F 2 "Package_QFP:LQFP-64_10x10mm_P0.5mm" H 1800 2300 50  0001 R CNN
@@
 Wire Wire Line
 	4800 2100 5500 2100
+$Comp
+L ASMB-KTF0-0A306:ASMB-KTF0-0A306 D2
+U 1 1 60B96BC3
+P 5700 5850
+F 0 "D2" H 5980 5946 50  0000 L CNN
+F 1 "ASMB-KTF0-0A306" H 5980 5855 50  0000 L CNN
+F 2 "LED_SMD:LED_ASMB-KTF0-0A306" H 5700 5850 50  0001 L BNN
+F 3 "" H 5700 5850 50  0001 L BNN
+F 4 "PLCC-4 Broadcom" H 5700 5850 50  0001 L BNN "PACKAGE"
+F 5 "Broadcom" H 5700 5850 50  0001 L BNN "MANUFACTURER"
+F 6 "Manufacturer recommendation" H 5700 5850 50  0001 L BNN "STANDARD"
+F 7 "15sep2017" H 5700 5850 50  0001 L BNN "PART_REV"
+F 8 "0.16 USD" H 5700 5850 50  0001 L BNN "PRICE"
+F 9 "Good" H 5700 5850 50  0001 L BNN "AVAILABILITY"
+F 10 "ASMB-KTF0-0A306" H 5700 5850 50  0001 L BNN "MP"
+F 11 "2220 Tricolor PLCC4 Surface Mount LED" H 5700 5850 50  0001 L BNN "DESCRIPTION"
+	1    5700 5850
+	1    0    0    -1
+$EndComp
+Wire Wire Line
+	5500 5950 5500 6050
+Wire Wire Line
+	5700 5950 5700 6100
+Wire Wire Line
+	5900 5950 5900 6050
+Wire Wire Line
+	5500 5500 5500 5550
+Wire Wire Line
+	5600 5550 5500 5550
+Connection ~ 5500 5550
+Wire Wire Line
+	5500 5550 5500 5650
+Text Notes 5400 5750 0    50   ~ 0
+R
+Text Notes 5650 5750 0    50   ~ 0
+B
+Text Notes 5850 5750 0    50   ~ 0
+G
+$Comp
+L FDV305N:FDV305N Q3
+U 1 1 60BC1078
+P 6050 6550
+F 0 "Q3" H 6258 6596 50  0000 L CNN
+F 1 "FDV305N" H 6258 6505 50  0000 L CNN
+F 2 "SOT95P240X111-3N" H 6050 6550 50  0001 L BNN
+F 3 "" H 6050 6550 50  0001 L BNN
+F 4 "IPC 7351B" H 6050 6550 50  0001 L BNN "STANDARD"
+F 5 "1.11 mm" H 6050 6550 50  0001 L BNN "MAXIMUM_PACKAGE_HEIGHT"
+F 6 "ON Semiconductor" H 6050 6550 50  0001 L BNN "MANUFACTURER"
+F 7 "30 Jan 2018" H 6050 6550 50  0001 L BNN "PARTREV"
+	1    6050 6550
+	1    0    0    -1
+$EndComp
+$Comp
+L FDV305N:FDV305N Q2
+U 1 1 60BC32FF
+P 5600 6850
+F 0 "Q2" H 5808 6896 50  0000 L CNN
+F 1 "FDV305N" H 5808 6805 50  0000 L CNN
+F 2 "SOT95P240X111-3N" H 5600 6850 50  0001 L BNN
+F 3 "" H 5600 6850 50  0001 L BNN
+F 4 "IPC 7351B" H 5600 6850 50  0001 L BNN "STANDARD"
+F 5 "1.11 mm" H 5600 6850 50  0001 L BNN "MAXIMUM_PACKAGE_HEIGHT"
+F 6 "ON Semiconductor" H 5600 6850 50  0001 L BNN "MANUFACTURER"
+F 7 "30 Jan 2018" H 5600 6850 50  0001 L BNN "PARTREV"
+	1    5600 6850
+	1    0    0    -1
+$EndComp
+$Comp
+L FDV305N:FDV305N Q1
+U 1 1 60BC3BA9
+P 5200 6550
+F 0 "Q1" H 5408 6596 50  0000 L CNN
+F 1 "FDV305N" H 5408 6505 50  0000 L CNN
+F 2 "SOT95P240X111-3N" H 5200 6550 50  0001 L BNN
+F 3 "" H 5200 6550 50  0001 L BNN
+F 4 "IPC 7351B" H 5200 6550 50  0001 L BNN "STANDARD"
+F 5 "1.11 mm" H 5200 6550 50  0001 L BNN "MAXIMUM_PACKAGE_HEIGHT"
+F 6 "ON Semiconductor" H 5200 6550 50  0001 L BNN "MANUFACTURER"
+F 7 "30 Jan 2018" H 5200 6550 50  0001 L BNN "PARTREV"
+	1    5200 6550
+	1    0    0    -1
+$EndComp
 $EndSCHEMATC

Commit message: ok
Parts:
- D2: symbol ASMB-KTF0-0A306:ASMB-KTF0-0A306 -> board-rescue:ASMB-KTF0-0A306-ASMB-KTF0-0A306
- Q1, Q2, Q3: symbol FDV305N:FDV305N -> board-rescue:FDV305N-FDV305N
Connections:
- net labels added: SWDCLK, SWDIO, SWO
- net labels removed: PGND1, PGND2, TPS_GND
- wire segments 145 -> 146
Changed lines of the file:
@@
 $EndComp
-Wire Wire Line
-	1800 6850 1650 6850
 Wire Wire Line
 	1650 6850 1650 6800
@@
 VFB1
 Text GLabel 6200 4150 0    50   Input ~ 0
-PGND1
+GND
 Text GLabel 6200 4000 0    50   Input ~ 0
 SW1
@@
 SW2
 Text GLabel 7050 4150 2    50   Input ~ 0
-PGND2
+GND
 Text GLabel 7050 4600 2    50   Input ~ 0
 VFB2
 Text GLabel 7850 3550 0    50   Input ~ 0
-PGND2
+GND
 Wire Wire Line
 	7150 4750 7050 4750
@@
 12V +/- 10%
 Text GLabel 6200 4750 0    50   Input ~ 0
-TPS_GND
+GND
 Text GLabel 5150 4100 2    50   Input ~ 0
-TPS_GND
+GND
 Text GLabel 6200 4300 0    50   Input ~ 0
 EN1_IN
@@
 SW1
 Text GLabel 5500 3500 2    50   Input ~ 0
-PGND1
+GND
 $Comp
 L power:GND #PWR017
@@
 	4800 2100 5500 2100
 $Comp
-L ASMB-KTF0-0A306:ASMB-KTF0-0A306 D2
+L board-rescue:ASMB-KTF0-0A306-ASMB-KTF0-0A306 D2
 U 1 1 60B96BC3
 P 5700 5850
@@
 G
 $Comp
-L FDV305N:FDV305N Q3
+L board-rescue:FDV305N-FDV305N Q3
 U 1 1 60BC1078
 P 6050 6550
@@
 $EndComp
 $Comp
-L FDV305N:FDV305N Q2
+L board-rescue:FDV305N-FDV305N Q2
 U 1 1 60BC32FF
 P 5600 6850
@@
 $EndComp
 $Comp
-L FDV305N:FDV305N Q1
+L board-rescue:FDV305N-FDV305N Q1
 U 1 1 60BC3BA9
 P 5200 6550
@@
 	1    0    0    -1
 $EndComp
+Wire Wire Line
+	1650 6850 1800 6850
+Wire Wire Line
+	1650 6850 1650 7000
+Connection ~ 1650 6850
+Text GLabel 3100 3700 2    50   Input ~ 0
+SWDIO
+Text GLabel 3100 3800 2    50   Input ~ 0
+SWDCLK
+Text GLabel 3100 4400 2    50   Input ~ 0
+SWO
 $EndSCHEMATC

Commit message: Push
Parts:
- removed C23: 10u, Capacitor_SMD:C_0603_1608Metric, symbol Device:C_Small
- removed R5: 124k, Resistor_SMD:R_0603_1608Metric, symbol Device:R_Small_US
- removed R6: 22k1, Resistor_SMD:R_0603_1608Metric, symbol Device:R_Small_US
- removed U2: TPS542941, Package_SO:HTSSOP-16-1EP_4.4x5mm_P0.65mm_EP3.4x5mm_Mask2.46x2.31mm_ThermalVias, symbol board-rescue:TPS542941
- added R1: 619k, Resistor_SMD:R_0402_1005Metric, symbol Device:R_Small_US
- added R2: 137k, Resistor_SMD:R_0402_1005Metric, symbol Device:R_Small_US
- added U2: LTC3622-23_5, Package_SO:MSOP-16-1EP_3x4mm_P0.5mm_EP1.65x2.85mm_ThermalVias, symbol board-rescue:LTC3622-23_5
- C15: value 22u -> 10u
- C16: value 10u -> 1u; footprint Capacitor_SMD:C_0603_1608Metric -> Capacitor_SMD:C_0402_1005Metric
- C18: value 100n -> 22p; footprint Capacitor_SMD:C_0603_1608Metric -> Capacitor_SMD:C_0402_1005Metric
- C21: value 1u -> 22u; footprint Capacitor_SMD:C_0603_1608Metric -> Capacitor_SMD:C_0402_1005Metric
- C22: value 100n -> 22u; footprint Capacitor_SMD:C_0603_1608Metric -> Capacitor_SMD:C_0402_1005Metric
- C24: value 22u -> 22p; footprint Capacitor_SMD:C_0603_1608Metric -> Capacitor_SMD:C_0402_1005Metric
- C5, C7: LSCS Part # (none) -> C32949
- F1: value 300mA -> 0ZCJ0050AF2E
- L1: value 4u7 -> 2u7
- L2: value 2u2 -> 3u3; LCSC Part # (none) -> C370336
- Q1, Q2, Q3: footprint SOT95P240X111-3N -> FDV305N:SOT95P240X111-3N
- R10: value 73k2 -> 619k; footprint Resistor_SMD:R_0603_1608Metric -> Resistor_SMD:R_0402_1005Metric
- R11: value 22k1 -> 84k5; footprint Resistor_SMD:R_0603_1608Metric -> Resistor_SMD:R_0402_1005Metric
- R3: LCSC Part # (none) -> C478874
- Y1: LCSC Part # (none) -> C13738
Connections:
- net VBST1 is gone; now on net +3V3: C18.1
- net VBST2 is gone; now on net +5V: C22.1
- net +12V: now also C15.1, C20.1, FB2.1, U2.1 (VIN1), U2.10 (RUN2), U2.14 (RUN1), U2.2 (SVIN), U2.8 (VIN2)
- net +3V3: now also C21.1, L1.2, R1.2; no longer C24.1, L2.2, R10.2
- net +5V: now also C24.1, L2.2, R10.2; no longer C15.1, L1.1
- net FLASH_!HOLD: now also U1.40 (PC9); no longer U1.38 (PC7)
- net FLASH_!WP: now also U1.39 (PC8); no longer U1.37 (PC6)
- net GND: now also C22.2, R2.1, U2.15 (NC), U2.5 (PHASE), U2.7 (ILIM); no longer C24.2
- net LCD_DB0: now also U1.24 (PC4); no longer U1.8 (PC0)
- net LCD_DB1: now also U1.25 (PC5); no longer U1.9 (PC1)
- net LCD_DB2: now also U1.26 (PB0); no longer U1.10 (PC2)
- net LCD_DB3: now also U1.28 (PB2); no longer U1.11 (PC3)
- net SPI2_!CS: now also U1.38 (PC7); no longer U1.33 (PB12)
- net SW1: now also L2.1, U2.16 (SW1); no longer C18.2, L1.2
- net SW2: now also L1.1, U2.9 (SW2); no longer C22.2, L2.1
- removed net BUCK_IN: C16.1, C20.1, FB2.1
- net VFB2 renamed FB1
- net FB1: now also C24.2, U2.13 (FB1)
- new net FB2: C18.2, R1.1, R2.2, U2.11 (FB2)
- new net INTVCC: C16.1, U2.12 (INTVCC), U2.4 (MODESYNC)
- no-connect marks 2 -> 21
Other:
- note added: "500mA hold\n"
- note added: "DO NOT STUFF\n"
- note added: "POW LED"
- note removed: "Fix enables\n"
- moved on the sheet: C24, R10, R11
