File: board/connectors.sch (KiCad schematic (older format))
At the start: 16 parts, among them J2 Conn_ARM_JTAG_SWD_10, J3 USB_B_Micro, J4 Conn_01x04_Male, J5 Screw_Terminal_01x02, U6 USBLC6-2SC6

Commit message: Push
Parts:
- added C?: 1u, Capacitor_SMD:C_0402_1005Metric, symbol Device:C_Small
- added C?: 4u7, Capacitor_SMD:C_0402_1005Metric, symbol Device:C_Small
- added C?: 100n, Capacitor_SMD:C_0402_1005Metric, symbol Device:C_Small
- added J?: Conn_01x16_Female, symbol Connector:Conn_01x16_Female
- added R5: 10k, Resistor_SMD:R_0603_1608Metric, symbol Device:R_Small_US
- added R?: 15k, Resistor_SMD:R_0603_1608Metric, symbol Device:R_Small_US
- added R?: 220, Resistor_SMD:R_0603_1608Metric, symbol Device:R_Small_US
- added SW1: SW_SPDT, Button_Switch_SMD:SW_SPDT_PCM12, symbol Switch:SW_SPDT
- added TP1: TestPoint, TestPoint:TestPoint_Pad_D1.0mm, symbol Connector:TestPoint
Connections:
- net +12V: now also J5.2 (Pin_2); no longer J5.1 (Pin_1)
- net +3V3: now also SW1.1 (A)
- net +5V: now also C?.1, C?.1, C?.1, J?.1 (Pin_1), R?.1, R?.1
- net GND: now also J5.1 (Pin_1), C?.2, C?.2, C?.2, J?.11 (Pin_11), J?.12 (Pin_12), J?.13 (Pin_13), J?.14 (Pin_14), J?.15 (Pin_15), J?.16 (Pin_16), J?.2 (Pin_2), J?.3 (Pin_3), R?.2, R?.2, SW1.3 (C); no longer J5.2 (Pin_2)
- new net: R5.1, SW1.2 (B)
- new net BOOT0: R5.2
- new net LCD_DB0: J?.7 (Pin_7)
- new net LCD_DB1: J?.8 (Pin_8)
- new net LCD_DB2: J?.9 (Pin_9)
- new net LCD_DB3: J?.10 (Pin_10)
- new net LCD_EN: J?.5 (Pin_5)
- new net LCD_RS: J?.4 (Pin_4)
- new net LCD_RW: J?.6 (Pin_6)
- new net RCC_MCO1: TP1.1
Other:
- note added: "Boot\n"
- note added: "LCD pins\n"
- moved on the sheet: J5

Commit message: Take 2
Connections:
- net VBUS: no longer J3.1 (VBUS)
- no-connect marks 3 -> 4
Changed lines of the file:
@@
 $EndDescr
-$Comp
-L Mechanical:MountingHole H1
-U 1 1 609E84AC
-P 5800 3500
-F 0 "H1" H 5900 3546 50  0000 L CNN
-F 1 "MountingHole" H 5900 3455 50  0000 L CNN
-F 2 "MountingHole:MountingHole_3.5mm_Pad_Via" H 5800 3500 50  0001 C CNN
-F 3 "~" H 5800 3500 50  0001 C CNN
-	1    5800 3500
-	1    0    0    -1
-$EndComp
 $Comp
 L Mechanical:MountingHole H3
@@
 $EndComp
 NoConn ~ 3900 2700
-$Comp
-L power:VBUS #PWR061
-U 1 1 60B231C0
-P 4400 1950
-F 0 "#PWR061" H 4400 1800 50  0001 C CNN
-F 1 "VBUS" H 4415 2123 50  0000 C CNN
-F 2 "" H 4400 1950 50  0001 C CNN
-F 3 "" H 4400 1950 50  0001 C CNN
-	1    4400 1950
-	1    0    0    -1
-$EndComp
-Wire Wire Line
-	4400 1950 4400 2100
-Wire Wire Line
-	4400 2100 4300 2100
 Text GLabel 4300 2300 2    50   Input ~ 0
 USB_CONN_D+
@@
 Wire Notes Line
 	8050 1350 10550 1350
+$Comp
+L Mechanical:MountingHole H1
+U 1 1 609E84AC
+P 5800 3500
+F 0 "H1" H 5900 3546 50  0000 L CNN
+F 1 "MountingHole" H 5900 3455 50  0000 L CNN
+F 2 "MountingHole:MountingHole_3.5mm_Pad_Via" H 5800 3500 50  0001 C CNN
+F 3 "~" H 5800 3500 50  0001 C CNN
+	1    5800 3500
+	1    0    0    -1
+$EndComp
+NoConn ~ 4300 2100
 $EndSCHEMATC
